Commit message: DiffDriveController applies radius to velocities

File: urdf/macros.xacro (robot description, xacro)
@@ -52,5 +52,5 @@
             <origin xyz="${tX*chassisLength/2} ${tY*wheelWidth/2+tY*chassisWidth/2} ${wheelRadius}" rpy="0 0 0" />
             <axis xyz="0 1 0" rpy="0 0 0" />
-            <limit effort="100" velocity="100"/>
+            <limit effort="1" velocity="${1/wheelRadius}"/>
             <joint_properties damping="0.0" friction="0.0"/>
         </joint>
